File: pcb/pcb_front/keys.sch (KiCad schematic (older format))
At the start: 303 parts

Commit message: Finish footprint assignments
Parts:
- D10, D100, D101, D102, D103, D104, D105, D106, D107, D11, D12, D13, D14, D15, D16, D17, D18, D19, D20, D21, D22, D23, D24, D25, D26, D27, D28, D29, D30, D31, D32, D33, D34, D35, D36, D37, D38, D39, D40, D41, D42, D43, D44, D45, D46, D47, D48, D49, D50, D51, D52, D53, D54, D55, D56, D57, D58, D59, D60, D61, D62, D63, D64, D65, D66, D67, D68, D69, D7, D70, D71, D72, D73, D74, D75, D76, D77, D78, D79, D8, D80, D81, D82, D83, D84, D85, D86, D87, D88, D89, D9, D90, D91, D92, D93, D94, D95, D96, D97, D98, D99: footprint (none) -> Diode_THT:D_DO-35_SOD27_P7.62mm_Horizontal
- MX1, MX10, MX101, MX11, MX12, MX13, MX14, MX15, MX16, MX17, MX18, MX19, MX2, MX20, MX21, MX22, MX23, MX24, MX25, MX26, MX27, MX28, MX3, MX30, MX31, MX32, MX33, MX34, MX36, MX37, MX38, MX39, MX4, MX40, MX41, MX42, MX43, MX44, MX45, MX46, MX47, MX48, MX5, MX50, MX51, MX52, MX53, MX56, MX57, MX58, MX59, MX6, MX60, MX61, MX62, MX63, MX64, MX65, MX66, MX68, MX69, MX7, MX70, MX71, MX73, MX74, MX75, MX76, MX77, MX78, MX79, MX8, MX80, MX81, MX82, MX84, MX85, MX86, MX87, MX88, MX9, MX94, MX95, MX96, MX97, MX98, MX99: footprint (none) -> MX_Only:MXOnly-1U
- MX100: footprint (none) -> MX_Only:MXOnly-2U-ReversedStabilizers
- MX29: footprint (none) -> MX_Only:MXOnly-2U
- MX35, MX49: footprint (none) -> MX_Only:MXOnly-1.5U
- MX54, MX89: footprint (none) -> MX_Only:MXOnly-2U-ReversedVerticalStabilizers
- MX55, MX83: footprint (none) -> MX_Only:MXOnly-1.75U
- MX67: footprint (none) -> MX_Only:MXOnly-2.25U-FLIPPED
- MX72: footprint (none) -> MX_Only:MXOnly-2.25U
- MX90, MX91, MX92: footprint (none) -> MX_Only:MXOnly-1.25U
- MX93: footprint (none) -> MX_Only:MXOnly-6.25U-ReversedStabilizers
- R100, R101, R102, R103, R104, R105, R106, R107, R108, R109, R110, R111, R112, R12, R13, R14, R15, R16, R17, R18, R19, R20, R21, R22, R23, R24, R25, R26, R27, R28, R29, R30, R31, R32, R33, R34, R35, R36, R37, R38, R39, R40, R41, R42, R43, R44, R45, R46, R47, R48, R49, R50, R51, R52, R53, R54, R55, R56, R57, R58, R59, R60, R61, R62, R63, R64, R65, R66, R67, R68, R69, R70, R71, R72, R73, R74, R75, R76, R77, R78, R79, R80, R81, R82, R83, R84, R85, R86, R87, R88, R89, R90, R91, R92, R93, R94, R95, R96, R97, R98, R99: footprint (none) -> Resistor_THT:R_Axial_DIN0204_L3.6mm_D1.6mm_P7.62mm_Horizontal
