File: pcb/pcb_front/main_pcb.kicad_pcb (KiCad board)
At the start: 2 copper layers, 334 parts, among them J1 AVR-ISP-6, J2 USB_C_Receptacle_USB2.0, Q1 Q_NMOS_DGS, SW1 RESET, SW2 BOOT, SW3 BL_STEP, U1 ATmega32-16PU, Y1 Crystal

Commit message: Begin PCB Layout
Parts:
- moved MX89 507.8 mm to (519.3, 275.4)
- moved MX100 496.6 mm to (471.7, 284.9)
- moved MX54 467.9 mm to (519.3, 237.3)
- moved MX34 440.2 mm to (519.3, 208.7)
- moved MX67 435.8 mm to (407.3, 246.8)
- moved MX101 427.8 mm to (500.2, 284.9)
- moved MX88 425.9 mm to (500.2, 265.9)
- moved MX86 420.4 mm to (462.2, 265.9)
- moved MX87 411.7 mm to (481.2, 265.9)
- moved MX29 388.7 mm to (409.6, 208.7)
- moved MX50 388.5 mm to (438.2, 227.8)
- moved MX93 387.4 mm to (273.9, 284.9)
- moved MX83 387.0 mm to (392.9, 265.9)
- moved MX85 374.6 mm to (438.2, 265.9)
- moved MX73 374.2 mm to (195.3, 265.9)
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