File: pcb/main_front/main_pcb.kicad_pcb (KiCad board)
At the start: 2 copper layers, 334 parts, among them J1 AVR-ISP-6, J2 USB_C_Receptacle_USB2.0, Q1 Q_NMOS_DGS, SW1 RESET, SW2 BOOT, SW3 BL_STEP, U1 ATmega32-16PU, Y1 Crystal

Commit message: Begin revised PCB layout
Parts:
- removed D106, D107, D37, D38, D39, D40, D57, D58, D59, D60, D75, D76, D77, D92, D93, D94, D95: 1N4148, Diode_THT:D_DO-35_SOD27_P7.62mm_Horizontal
- removed D2: NUMLOCK, LED_THT:LED_D3.0mm_Clear
- removed MX100: MX-LED, MX_Only:MXOnly-2U-ReversedStabilizers
- removed MX101, MX31, MX32, MX33, MX34, MX51, MX52, MX53, MX69, MX70, MX71, MX86, MX87, MX88: MX-LED, MX_Only:MXOnly-1U
- removed MX54, MX89: MX-LED, MX_Only:MXOnly-2U-ReversedVerticalStabilizers
- removed R100, R111, R112, R42, R43, R44, R45, R62, R63, R64, R65, R80, R81, R82, R97, R98, R99: 470, Resistor_THT:R_Axial_DIN0204_L3.6mm_D1.6mm_P7.62mm_Horizontal
- removed R9: 1.5k, Resistor_THT:R_Axial_DIN0204_L3.6mm_D1.6mm_P7.62mm_Horizontal
- added J3: Conn_01x16_Male, Connector_PinHeader_2.54mm:PinHeader_2x08_P2.54mm_Horizontal, F.Cu at (300.9, -75.1)

Commit message: Finish rough Resistor and Diode layout
Parts:
- J2: footprint Connector_USB:USB_C_Receptacle_GCT_USB4085 -> keyboard_parts:USB_C_GCT_USB4085
- moved R12 317.2 mm to (145.5, 143.5), turned to 90 degrees
- moved U1 305.3 mm to (371.5, 173.5), turned to 90 degrees
- moved R13 305.3 mm to (168.0, 149.8), turned to 90 degrees
- moved D61 299.6 mm to (153.5, 166.0), turned to 270 degrees
- moved D11 285.6 mm to (208.5, 160.0), turned to 270 degrees
- moved R101 281.9 mm to (158.0, 153.5), turned to 90 degrees
- moved R84 280.7 mm to (178.0, 145.8), turned to 90 degrees
- moved D12 280.2 mm to (221.0, 160.0), turned to 270 degrees
- moved D20 271.4 mm to (336.0, 162.0), turned to 270 degrees
- moved D8 271.1 mm to (168.5, 168.0), turned to 270 degrees
- moved D67 267.2 mm to (243.5, 168.0), turned to 270 degrees
- moved J3 267.1 mm to (434.7, 156.0)
- moved D41 266.2 mm to (151.0, 164.0), turned to 270 degrees
- moved D90 261.6 mm to (331.0, 167.5), turned to 270 degrees
- moved D42 259.3 mm to (163.5, 164.0), turned to 270 degrees
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Other:
- board outline added: 304.9 x 167.1 mm

Commit message: Continue PCB Layout
Parts:
- added REF**: MountingHole_2.2mm_M2_Pad, MountingHole:MountingHole_2.2mm_M2_Pad, F.Cu at (344.8, 176.2)
- added REF**: MountingHole_2.2mm_M2_Pad, MountingHole:MountingHole_2.2mm_M2_Pad, F.Cu at (344.8, 138.8)
- added REF**: MountingHole_2.2mm_M2_Pad, MountingHole:MountingHole_2.2mm_M2_Pad, F.Cu at (247.0, 176.2)
- added REF**: MountingHole_2.2mm_M2_Pad, MountingHole:MountingHole_2.2mm_M2_Pad, F.Cu at (247.0, 138.8)
- added REF**: MountingHole_2.2mm_M2_Pad, MountingHole:MountingHole_2.2mm_M2_Pad, F.Cu at (147.0, 176.2)
- added REF**: MountingHole_2.2mm_M2_Pad, MountingHole:MountingHole_2.2mm_M2_Pad, F.Cu at (443.8, 176.2)
- added REF**: MountingHole_2.2mm_M2_Pad, MountingHole:MountingHole_2.2mm_M2_Pad, F.Cu at (443.8, 138.8)
- added REF**: MountingHole_2.2mm_M2_Pad, MountingHole:MountingHole_2.2mm_M2_Pad, F.Cu at (147.0, 138.8)
- moved Y1 334.4 mm to (401.4, 170.8)
- moved C4 315.7 mm to (411.4, 171.8), turned to 90 degrees
- moved R7 293.2 mm to (369.9, 146.3), turned to 180 degrees
- moved R5 292.7 mm to (369.9, 156.8), turned to 180 degrees
- moved R3 292.5 mm to (369.9, 153.3), turned to 180 degrees
- moved R10 290.8 mm to (369.9, 160.3), turned to 180 degrees
- moved R8 285.8 mm to (369.9, 149.8), turned to 180 degrees
- moved R11 285.5 mm to (362.3, 163.8)
- moved J1 282.5 mm to (364.4, 168.3)
- moved Q1 280.0 mm to (380.9, 138.4), turned to 270 degrees
- moved R1 279.7 mm to (376.8, 144.8), turned to 90 degrees
- moved R2 279.3 mm to (373.7, 144.8), turned to 90 degrees
- moved R4 277.6 mm to (369.9, 142.8), turned to 180 degrees
- moved D6 268.4 mm to (369.9, 135.8), turned to 180 degrees
- moved R6 267.5 mm to (362.3, 139.3)
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Connections:
- U1 pad 20: col11 -> BOOT
- U1 pad 21: BOOT -> col11
Other:
- board size 304.9 x 167.1 mm -> 304.8 x 160.2 mm

Commit message: Added copper planes
Parts:
- moved C4 6.02 mm to (417.4, 171.3)
- moved Y1 5.52 mm to (406.9, 170.3)
- moved C5 5.02 mm to (401.4, 171.3)
- moved D6 1.12 mm to (368.9, 136.3)
- moved R10 1.12 mm to (368.9, 160.8)
- moved R11 1.12 mm to (361.3, 164.3)
- moved R3 1.12 mm to (368.9, 153.8)
- moved R4 1.12 mm to (368.9, 143.3)
- moved R5 1.12 mm to (368.9, 157.3)
- moved R6 1.12 mm to (361.3, 139.8)
- moved R7 1.12 mm to (368.9, 146.8)
- moved R8 1.12 mm to (368.9, 150.3)
Routing:
- added copper zone on B.Cu, net +5V
- added copper zone on F.Cu, net GND
- added copper zone on B.Cu, net LEDGND
Other:
- net class PWR added: clearance 0.2, trace_width 0.5, via_dia 0.8, via_drill 0.4
Changed lines of the file:
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@@
     (add_net row5)
   )
+  (net_class PWR ""
+    (clearance 0.2)
+    (trace_width 0.5)
+    (via_dia 0.8)
+    (via_drill 0.4)
+    (uvia_dia 0.3)
+    (uvia_drill 0.1)
+  )
   (module MountingHole:MountingHole_2.2mm_M2_Pad (layer F.Cu)
     (at 344.8 176.204)
@@
   )
   (module Crystal:Crystal_HC49-4H_Vertical (layer F.Cu)
-    (at 401.4 170.8)
+    (at 406.9 170.3)
     (descr "Crystal THT HC-49-4H http://5hertz.com/pdfs/04404_D.pdf")
     (tags "THT crystalHC-49-4H")
@@
   )
   (module Resistor_THT:R_Axial_DIN0204_L3.6mm_D1.6mm_P7.62mm_Horizontal (layer F.Cu)
-    (at 362.28 163.8)
+    (at 361.28 164.3)
     (descr "Resistor, Axial_DIN0204 series, Axial, Horizontal, pin pitch=7.62mm, 0.167W, length*diameter=3.6*1.6mm^2, http://cdn-reichelt.de/documents/datenblatt/B400/1_4W%23YAG.pdf")
     (tags "Resistor Axial_DIN0204 series Axial Horizontal pin pitch 7.62mm 0.167W length 3.6mm diameter 1.6mm")
@@
   )
   (module Resistor_THT:R_Axial_DIN0204_L3.6mm_D1.6mm_P7.62mm_Horizontal (layer F.Cu)
-    (at 369.9 160.3 180)
+    (at 368.9 160.8 180)
     (descr "Resistor, Axial_DIN0204 series, Axial, Horizontal, pin pitch=7.62mm, 0.167W, length*diameter=3.6*1.6mm^2, http://cdn-reichelt.de/documents/datenblatt/B400/1_4W%23YAG.pdf")
     (tags "Resistor Axial_DIN0204 series Axial Horizontal pin pitch 7.62mm 0.167W length 3.6mm diameter 1.6mm")
@@
   )
   (module Resistor_THT:R_Axial_DIN0204_L3.6mm_D1.6mm_P7.62mm_Horizontal (layer F.Cu)
-    (at 369.9 149.8 180)
+    (at 368.9 150.3 180)
     (descr "Resistor, Axial_DIN0204 series, Axial, Horizontal, pin pitch=7.62mm, 0.167W, length*diameter=3.6*1.6mm^2, http://cdn-reichelt.de/documents/datenblatt/B400/1_4W%23YAG.pdf")
     (tags "Resistor Axial_DIN0204 series Axial Horizontal pin pitch 7.62mm 0.167W length 3.6mm diameter 1.6mm")
@@
   )
   (module Resistor_THT:R_Axial_DIN0204_L3.6mm_D1.6mm_P7.62mm_Horizontal (layer F.Cu)
-    (at 369.9 146.3 180)
+    (at 368.9 146.8 180)
     (descr "Resistor, Axial_DIN0204 series, Axial, Horizontal, pin pitch=7.62mm, 0.167W, length*diameter=3.6*1.6mm^2, http://cdn-reichelt.de/documents/datenblatt/B400/1_4W%23YAG.pdf")
     (tags "Resistor Axial_DIN0204 series Axial Horizontal pin pitch 7.62mm 0.167W length 3.6mm diameter 1.6mm")
@@
   )
   (module Resistor_THT:R_Axial_DIN0204_L3.6mm_D1.6mm_P7.62mm_Horizontal (layer F.Cu)
-    (at 362.28 139.3)
+    (at 361.28 139.8)
     (descr "Resistor, Axial_DIN0204 series, Axial, Horizontal, pin pitch=7.62mm, 0.167W, length*diameter=3.6*1.6mm^2, http://cdn-reichelt.de/documents/datenblatt/B400/1_4W%23YAG.pdf")
     (tags "Resistor Axial_DIN0204 series Axial Horizontal pin pitch 7.62mm 0.167W length 3.6mm diameter 1.6mm")
@@
   )
   (module Resistor_THT:R_Axial_DIN0204_L3.6mm_D1.6mm_P7.62mm_Horizontal (layer F.Cu)
-    (at 369.9 156.8 180)
+    (at 368.9 157.3 180)
     (descr "Resistor, Axial_DIN0204 series, Axial, Horizontal, pin pitch=7.62mm, 0.167W, length*diameter=3.6*1.6mm^2, http://cdn-reichelt.de/documents/datenblatt/B400/1_4W%23YAG.pdf")
     (tags "Resistor Axial_DIN0204 series Axial Horizontal pin pitch 7.62mm 0.167W length 3.6mm diameter 1.6mm")
@@
   )
   (module Resistor_THT:R_Axial_DIN0204_L3.6mm_D1.6mm_P7.62mm_Horizontal (layer F.Cu)
-    (at 369.9 142.8 180)
+    (at 368.9 143.3 180)
     (descr "Resistor, Axial_DIN0204 series, Axial, Horizontal, pin pitch=7.62mm, 0.167W, length*diameter=3.6*1.6mm^2, http://cdn-reichelt.de/documents/datenblatt/B400/1_4W%23YAG.pdf")
     (tags "Resistor Axial_DIN0204 series Axial Horizontal pin pitch 7.62mm 0.167W length 3.6mm diameter 1.6mm")
@@
   )
   (module Resistor_THT:R_Axial_DIN0204_L3.6mm_D1.6mm_P7.62mm_Horizontal (layer F.Cu)
-    (at 369.9 153.3 180)
+    (at 368.9 153.8 180)
     (descr "Resistor, Axial_DIN0204 series, Axial, Horizontal, pin pitch=7.62mm, 0.167W, length*diameter=3.6*1.6mm^2, http://cdn-reichelt.de/documents/datenblatt/B400/1_4W%23YAG.pdf")
     (tags "Resistor Axial_DIN0204 series Axial Horizontal pin pitch 7.62mm 0.167W length 3.6mm diameter 1.6mm")
@@
   )
   (module Diode_THT:D_DO-35_SOD27_P7.62mm_Horizontal (layer F.Cu)
-    (at 369.9 135.8 180)
+    (at 368.9 136.3 180)
     (descr "Diode, DO-35_SOD27 series, Axial, Horizontal, pin pitch=7.62mm, , length*diameter=4*2mm^2, , http://www.diodes.com/_files/packages/DO-35.pdf")
     (tags "Diode DO-35_SOD27 series Axial Horizontal pin pitch 7.62mm  length 4mm diameter 2mm")
@@
   )
   (module Capacitor_THT:C_Disc_D3.0mm_W1.6mm_P2.50mm (layer F.Cu)
-    (at 396.4 171.8 90)
+    (at 401.4 171.3 90)
     (descr "C, Disc series, Radial, pin pitch=2.50mm, , diameter*width=3.0*1.6mm^2, Capacitor, http://www.vishay.com/docs/45233/krseries.pdf")
     (tags "C Disc series Radial pin pitch 2.50mm  diameter 3.0mm width 1.6mm Capacitor")
@@
   )
   (module Capacitor_THT:C_Disc_D3.0mm_W1.6mm_P2.50mm (layer F.Cu)
-    (at 411.4 171.8 90)
+    (at 417.4 171.3 90)
     (descr "C, Disc series, Radial, pin pitch=2.50mm, , diameter*width=3.0*1.6mm^2, Capacitor, http://www.vishay.com/docs/45233/krseries.pdf")
     (tags "C Disc series Radial pin pitch 2.50mm  diameter 3.0mm width 1.6mm Capacitor")
@@
   (gr_line (start 444.7032 294.386) (end 145.9992 294.386) (layer Edge.Cuts) (width 0.05))
   (gr_line (start 447.8 134.2) (end 447.7004 291.3888) (layer Edge.Cuts) (width 0.05))
+  (zone (net 1) (net_name GND) (layer F.Cu) (hatch edge 0.508)
+    (connect_pads (clearance 0.508))
+    (min_thickness 0.254)
+    (fill yes (arc_segments 32) (thermal_gap 0.508) (thermal_bridge_width 0.508))
+    (polygon
+      (pts
+        (xy 448.9 295.3) (xy 140.4 295.3) (xy 140.4 133.3) (xy 448.9 133.3)
+      )
+    )
+  )
+  (zone (net 2) (net_name +5V) (layer B.Cu) (hatch edge 0.508)
+    (connect_pads (clearance 0.508))
+    (min_thickness 0.254)
+    (fill yes (arc_segments 32) (thermal_gap 0.508) (thermal_bridge_width 0.508))
+    (polygon
+      (pts
+        (xy 368.9 176.3) (xy 146.9 176.3) (xy 146.9 138.8) (xy 368.9 138.8)
+      )
+    )
+  )
+  (zone (net 111) (net_name LEDGND) (layer B.Cu) (hatch edge 0.508)
+    (connect_pads (clearance 0.508))
+    (min_thickness 0.254)
+    (fill yes (arc_segments 32) (thermal_gap 0.508) (thermal_bridge_width 0.508))
+    (polygon
+      (pts
+        (xy 448.9 295.3) (xy 140.4 295.3) (xy 140.4 179.3) (xy 448.9 179.3)
+      )
+    )
+  )
 )

Commit message: removed some silk screens, added some, moved stuff around
Parts:
- moved Q1 20.0 mm to (380.9, 158.4)
- moved R1 20.0 mm to (376.8, 164.8)
- moved R2 20.0 mm to (373.7, 164.8)
- moved D1 19.1 mm to (423.4, 157.8)
- moved C4 12.0 mm to (418.4, 159.3)
- moved C5 12.0 mm to (402.4, 159.3)
- moved U1 12.0 mm to (375.1, 152.1)
- moved Y1 12.0 mm to (407.9, 158.3)
- moved R101 4.00 mm to (160.9, 155.8)
- moved R102 4.00 mm to (168.4, 155.8)
- moved R103 4.00 mm to (183.4, 155.8)
- moved R104 4.00 mm to (235.9, 155.8)
- moved R105 4.00 mm to (275.9, 151.8)
- moved R106 4.00 mm to (290.9, 151.8)
- moved R107 4.00 mm to (305.9, 151.8)
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
Commit message: adjusted edge cuts to be square
Parts:
- moved SW3 8.80 mm to (167.4, 136.8)
Other:
- outline, holes or cut-outs redrawn
Changed lines of the file:
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@@
   (general
     (thickness 1.6)
-    (drawings 20)
+    (drawings 19)
     (tracks 0)
     (zones 0)
@@
     (mod_text_size 1 1)
     (mod_text_width 0.15)
-    (pad_size 1.524 1.524)
-    (pad_drill 0.762)
+    (pad_size 4.4 4.4)
+    (pad_drill 2.2)
     (pad_to_mask_clearance 0.051)
     (solder_mask_min_width 0.25)
@@
       (effects (font (size 1 1) (thickness 0.15)))
     )
-    (pad 1 thru_hole circle (at 0 0) (size 4.4 4.4) (drill 2.2) (layers *.Cu *.Mask))
+    (pad 1 thru_hole circle (at 0 -0.004) (size 4.4 4.4) (drill 2.2) (layers *.Cu *.Mask))
   )
   (module MountingHole:MountingHole_2.2mm_M2_Pad (layer F.Cu)
@@
       (effects (font (size 1 1) (thickness 0.15)))
     )
-    (pad 1 thru_hole circle (at 0 0) (size 4.4 4.4) (drill 2.2) (layers *.Cu *.Mask))
+    (pad 1 thru_hole circle (at 0 -0.008) (size 4.4 4.4) (drill 2.2) (layers *.Cu *.Mask))
   )
   (module MountingHole:MountingHole_2.2mm_M2_Pad (layer F.Cu)
@@
       (effects (font (size 1 1) (thickness 0.15)))
     )
-    (pad 1 thru_hole circle (at 0 0) (size 4.4 4.4) (drill 2.2) (layers *.Cu *.Mask))
+    (pad 1 thru_hole circle (at 0 -0.204) (size 4.4 4.4) (drill 2.2) (layers *.Cu *.Mask))
   )
   (module MountingHole:MountingHole_2.2mm_M2_Pad (layer F.Cu)
@@
       (effects (font (size 1 1) (thickness 0.15)))
     )
-    (pad 1 thru_hole circle (at 0 0) (size 4.4 4.4) (drill 2.2) (layers *.Cu *.Mask))
+    (pad 1 thru_hole circle (at 0 -0.008) (size 4.4 4.4) (drill 2.2) (layers *.Cu *.Mask))
   )
   (module keyboard_parts:USB_C_GCT_USB4085 (layer F.Cu)
@@
       (effects (font (size 1 1) (thickness 0.15)))
     )
-    (pad 1 thru_hole circle (at 0 0) (size 4.4 4.4) (drill 2.2) (layers *.Cu *.Mask))
+    (pad 1 thru_hole circle (at 0 -0.004) (size 4.4 4.4) (drill 2.2) (layers *.Cu *.Mask))
   )
   (module MountingHole:MountingHole_2.2mm_M2_Pad (layer F.Cu)
@@
       (effects (font (size 1 1) (thickness 0.15)))
     )
-    (pad 1 thru_hole circle (at 0 0) (size 4.4 4.4) (drill 2.2) (layers *.Cu *.Mask))
+    (pad 1 thru_hole circle (at 0 -0.004) (size 4.4 4.4) (drill 2.2) (layers *.Cu *.Mask))
   )
   (module Connector_PinHeader_2.54mm:PinHeader_2x08_P2.54mm_Horizontal (layer F.Cu)
@@
   )
   (module Button_Switch_THT:SW_Tactile_SPST_Angled_PTS645Vx31-2LFS (layer F.Cu)
-    (at 158.6 136.8)
+    (at 167.4 136.8)
     (descr "tactile switch SPST right angle, PTS645VL31-2 LFS")
     (tags "tactile switch SPST angled PTS645VL31-2 LFS C&K Button")
@@
     (arrow2b (pts (xy 142.94375 307.2) (xy 144.070254 306.613579)))
   )
-  (gr_arc (start 444.7032 291.3888) (end 444.7032 294.386) (angle -90) (layer Edge.Cuts) (width 0.05))
-  (gr_arc (start 146 137.2) (end 146 134.2028) (angle -90) (layer Edge.Cuts) (width 0.05))
-  (gr_arc (start 145.9992 291.3888) (end 143.002 291.3888) (angle -90) (layer Edge.Cuts) (width 0.05))
-  (gr_line (start 447.8 134.2028) (end 146 134.2028) (layer Edge.Cuts) (width 0.05))
-  (gr_line (start 143.002 291.3888) (end 143.0028 137.2) (layer Edge.Cuts) (width 0.05))
-  (gr_line (start 444.7032 294.386) (end 145.9992 294.386) (layer Edge.Cuts) (width 0.05))
-  (gr_line (start 447.8 134.2) (end 447.7004 291.3888) (layer Edge.Cuts) (width 0.05))
+  (gr_arc (start 146 137.2) (end 146 134.2) (angle -90) (layer Edge.Cuts) (width 0.05))
+  (gr_arc (start 145.9972 291.4) (end 143 291.4) (angle -90) (layer Edge.Cuts) (width 0.05))
+  (gr_line (start 447.8 134.2) (end 146 134.2) (layer Edge.Cuts) (width 0.05))
+  (gr_line (start 143 291.4) (end 143 137.2) (layer Edge.Cuts) (width 0.05))
+  (gr_line (start 447.8 294.4) (end 146 294.4) (layer Edge.Cuts) (width 0.05))
+  (gr_line (start 447.8 134.2) (end 447.8 294.4) (layer Edge.Cuts) (width 0.05))
   (zone (net 1) (net_name GND) (layer F.Cu) (hatch edge 0.508)
     (connect_pads (clearance 0.508))
