File: pcb/main_front/main_pcb.kicad_pcb (KiCad board)
At the start: 2 copper layers, 304.8 x 160.2 mm, 296 parts, among them J1 AVR-ISP-6, J2 USB_C_Receptacle_USB2.0, J3 Conn_01x16_Male, Q1 Q_NMOS_DGS, SW1 RESET, SW2 BOOT, SW3 BL_STEP, U1 ATmega32-16PU, Y1 Crystal

Commit message: Finish routing main PCB
Parts:
- moved R8 40.7 mm to (247.2, 61.3)
- moved R7 38.8 mm to (247.2, 64.8)
- moved R10 17.8 mm to (285.4, 68.0)
- moved R4 10.5 mm to (285.4, 78.8)
- moved D3 3.60 mm to (226.2, 61.3)
- moved D4 3.60 mm to (226.2, 64.9)
- moved R3 3.50 mm to (285.4, 82.3)
- moved R5 3.50 mm to (285.4, 85.8)
- moved C4 0.75 mm to (335.9, 85.0)
- moved C5 0.75 mm to (319.9, 85.0)
- moved Y1 0.75 mm to (325.4, 84.0)
Routing:
- net LEDGND: track 40.1 -> 2262.2 mm, vias 0 -> 8
- net col2: track 108.1 -> 549.7 mm, vias 0 -> 22
- net col5: track 86.1 -> 512.0 mm, vias 0 -> 22
- net col3: track 86.1 -> 452.9 mm, vias 0 -> 28
- net col4: track 86.1 -> 452.8 mm, vias 0 -> 26
- net col6: track 106.1 -> 471.5 mm, vias 0 -> 18
- net col8: track 86.1 -> 427.8 mm, vias 0 -> 1
- net row4: track 0.00 -> 327.6 mm, vias 0 -> 3
- net col1: track 98.3 -> 418.3 mm, vias 0 -> 2
- net row0: track 0.00 -> 315.2 mm, vias 0 -> 3
- net row3: track 0.00 -> 314.1 mm, vias 0 -> 3
- net row1: track 0.00 -> 309.4 mm, vias 0 -> 3
- net row2: track 0.00 -> 307.8 mm, vias 0 -> 3
- net row5: track 0.00 -> 300.0 mm, vias 0 -> 4
- net col7: track 86.1 -> 365.1 mm, vias 0 -> 20
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
Commit message: Freerouting work
Parts:
- removed REF** (x12): MountingHole_2.2mm_M2_Pad, MountingHole:MountingHole_2.2mm_M2_Pad
- added MOUNT10: MountingHole_2.2mm_M2_Pad, MountingHole:MountingHole_2.2mm_M2_Pad, F.Cu at (211.8, 124.2)
- added MOUNT11: MountingHole_2.2mm_M2_Pad, MountingHole:MountingHole_2.2mm_M2_Pad, F.Cu at (345.2, 124.2)
- added MOUNT12: MountingHole_2.2mm_M2_Pad, MountingHole:MountingHole_2.2mm_M2_Pad, F.Cu at (83.2, 209.9)
- added MOUNT13: MountingHole_2.2mm_M2_Pad, MountingHole:MountingHole_2.2mm_M2_Pad, F.Cu at (216.6, 210.0)
- added MOUNT14: MountingHole_2.2mm_M2_Pad, MountingHole:MountingHole_2.2mm_M2_Pad, F.Cu at (345.2, 200.3)
- added MOUNT2: MountingHole_2.2mm_M2_Pad, MountingHole:MountingHole_2.2mm_M2_Pad, F.Cu at (160.5, 63.2)
- added MOUNT3: MountingHole_2.2mm_M2_Pad, MountingHole:MountingHole_2.2mm_M2_Pad, F.Cu at (264.3, 63.2)
- added MOUNT4: MountingHole_2.2mm_M2_Pad, MountingHole:MountingHole_2.2mm_M2_Pad, F.Cu at (360.3, 63.2)
- added MOUNT5: MountingHole_2.2mm_M2_Pad, MountingHole:MountingHole_2.2mm_M2_Pad, F.Cu at (63.5, 101.2)
- added MOUNT7: MountingHole_2.2mm_M2_Pad, MountingHole:MountingHole_2.2mm_M2_Pad, F.Cu at (264.3, 101.2)
- added MOUNT8: MountingHole_2.2mm_M2_Pad, MountingHole:MountingHole_2.2mm_M2_Pad, F.Cu at (360.3, 101.2)
- added MOUNT9: MountingHole_2.2mm_M2_Pad, MountingHole:MountingHole_2.2mm_M2_Pad, F.Cu at (78.5, 124.1)
- renumbered REF** to MOUNT1, REF** to MOUNT6
Changed lines of the file:
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@@
     (tags "mounting hole 2.2mm m2")
     (attr virtual)
-    (fp_text reference REF** (at 0 -3.2) (layer F.SilkS) hide
+    (fp_text reference MOUNT6 (at 0 -3.2) (layer F.SilkS) hide
       (effects (font (size 1 1) (thickness 0.15)))
     )
@@
     (tags "mounting hole 2.2mm m2")
     (attr virtual)
-    (fp_text reference REF** (at 0 -3.2) (layer F.SilkS) hide
+    (fp_text reference MOUNT13 (at 0 -3.2) (layer F.SilkS) hide
       (effects (font (size 1 1) (thickness 0.15)))
     )
@@
     (tags "mounting hole 2.2mm m2")
     (attr virtual)
-    (fp_text reference REF** (at 0 -3.2) (layer F.SilkS) hide
+    (fp_text reference MOUNT10 (at 0 -3.2) (layer F.SilkS) hide
       (effects (font (size 1 1) (thickness 0.15)))
     )
@@
     (tags "mounting hole 2.2mm m2")
     (attr virtual)
-    (fp_text reference REF** (at 0 -3.2) (layer F.SilkS) hide
+    (fp_text reference MOUNT9 (at 0 -3.2) (layer F.SilkS) hide
       (effects (font (size 1 1) (thickness 0.15)))
     )
@@
     (tags "mounting hole 2.2mm m2")
     (attr virtual)
-    (fp_text reference REF** (at 0 -3.2) (layer F.SilkS) hide
+    (fp_text reference MOUNT11 (at 0 -3.2) (layer F.SilkS) hide
       (effects (font (size 1 1) (thickness 0.15)))
     )
@@
     (tags "mounting hole 2.2mm m2")
     (attr virtual)
-    (fp_text reference REF** (at 0 -3.2) (layer F.SilkS) hide
+    (fp_text reference MOUNT14 (at 0 -3.2) (layer F.SilkS) hide
       (effects (font (size 1 1) (thickness 0.15)))
     )
@@
     (tags "mounting hole 2.2mm m2")
     (attr virtual)
-    (fp_text reference REF** (at 0 -3.2) (layer F.SilkS) hide
+    (fp_text reference MOUNT12 (at 0 -3.2) (layer F.SilkS) hide
       (effects (font (size 1 1) (thickness 0.15)))
     )
@@
     (tags "mounting hole 2.2mm m2")
     (attr virtual)
-    (fp_text reference REF** (at 0 -3.2) (layer F.SilkS) hide
+    (fp_text reference MOUNT7 (at 0 -3.2) (layer F.SilkS) hide
       (effects (font (size 1 1) (thickness 0.15)))
     )
@@
     (tags "mounting hole 2.2mm m2")
     (attr virtual)
-    (fp_text reference REF** (at 0 -3.2) (layer F.SilkS) hide
+    (fp_text reference MOUNT3 (at 0 -3.2) (layer F.SilkS) hide
       (effects (font (size 1 1) (thickness 0.15)))
     )
@@
     (tags "mounting hole 2.2mm m2")
     (attr virtual)
-    (fp_text reference REF** (at 0 -3.2) (layer F.SilkS) hide
+    (fp_text reference MOUNT2 (at 0 -3.2) (layer F.SilkS) hide
       (effects (font (size 1 1) (thickness 0.15)))
     )
@@
     (tags "mounting hole 2.2mm m2")
     (attr virtual)
-    (fp_text reference REF** (at 0 -3.2) (layer F.SilkS) hide
+    (fp_text reference MOUNT5 (at 0 -3.2) (layer F.SilkS) hide
       (effects (font (size 1 1) (thickness 0.15)))
     )
@@
     (tags "mounting hole 2.2mm m2")
     (attr virtual)
-    (fp_text reference REF** (at 0 -3.2) (layer F.SilkS) hide
+    (fp_text reference MOUNT8 (at 0 -3.2) (layer F.SilkS) hide
       (effects (font (size 1 1) (thickness 0.15)))
     )
@@
     (tags "mounting hole 2.2mm m2")
     (attr virtual)
-    (fp_text reference REF** (at 0 -3.2) (layer F.SilkS) hide
+    (fp_text reference MOUNT4 (at 0 -3.2) (layer F.SilkS) hide
       (effects (font (size 1 1) (thickness 0.15)))
     )
@@
     (tags "mounting hole 2.2mm m2")
     (attr virtual)
-    (fp_text reference REF** (at 0 -3.2) (layer F.SilkS) hide
-      (effects (font (size 1 1) (thickness 0.15)))
-    )
+    (fp_text reference MOUNT1 (at 0 -3.2) (layer F.SilkS) hide
+      (effects (font (size 1 1) (thickness 0.15)))
+    )

Commit message: Finish PCB Silkscreen Decor
Parts:
- added REF**: OSHW-Logo2_14.6x12mm_SilkScreen, Symbol:OSHW-Logo2_14.6x12mm_SilkScreen, F.Cu at (334.3, 95.0)
- added REF**: ESD-Logo_8.9x8mm_SilkScreen, Symbol:ESD-Logo_8.9x8mm_SilkScreen, F.Cu at (320.7, 93.8)
Other:
- board text added: "JLCJLCJLCJLC"
- board text added: "QBoard rev0 By QuantumManiac and Jlsajfj 2021-08-30 Main Board"

Commit message: Fix wrong pinout on MOSFET
Parts:
- J2: footprint keyboard_parts:USB_C_GCT_USB4085 -> Connector_USB:USB_C_Receptacle_GCT_USB4085
- Q1: value Q_NMOS_DGS -> Q_NMOS_GDS
Connections:
- Q1 pad 1: LEDGND -> Net-(Q1-Pad1)
- Q1 pad 2: Net-(Q1-Pad2) -> LEDGND
- R1 pad 1: Net-(Q1-Pad2) -> Net-(Q1-Pad1)
- R2 pad 1: Net-(Q1-Pad2) -> Net-(Q1-Pad1)
- U1 pad 20: BOOT -> col11
- U1 pad 21: col11 -> BOOT
Routing:
- net Net-(Q1-Pad1): track 0.00 -> 12.8 mm
- net Net-(Q1-Pad2): track 10.2 -> 0.00 mm
- net LEDGND: track 2262.2 -> 2261.1 mm

Commit message: Fix USB footprint
Parts:
- J2: footprint Connector_USB:USB_C_Receptacle_GCT_USB4085 -> keyboard_parts:USB_C_GCT_USB4085
- moved Q1 0.11 mm to (297.5, 83.4)

Commit message: Fix pin issue in schematic and netlist
Connections:
- U1 pad 20: col11 -> BOOT
- U1 pad 21: BOOT -> col11
Routing:
- net Net-(Q1-Pad1): track 12.8 -> 12.2 mm
Changed lines of the file:
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@@
       (net 12 row0))
     (pad 20 thru_hole oval (at 0 48.26 90) (size 1.6 1.6) (drill 0.8) (layers *.Cu *.Mask)
-      (net 130 col11))
+      (net 216 BOOT))
     (pad 39 thru_hole oval (at 15.24 2.54 90) (size 1.6 1.6) (drill 0.8) (layers *.Cu *.Mask)
       (net 29 row1))
@@
       (net 141 col1))
     (pad 21 thru_hole oval (at 15.24 48.26 90) (size 1.6 1.6) (drill 0.8) (layers *.Cu *.Mask)
-      (net 216 BOOT))
+      (net 130 col11))
     (pad 1 thru_hole rect (at 0 0 90) (size 1.6 1.6) (drill 0.8) (layers *.Cu *.Mask)
       (net 113 col0))
@@
   (segment (start 74.0725 214.98) (end 72.62 214.98) (width 0.5) (layer F.Cu) (net 111))
   (segment (start 77.1425 218.05) (end 74.0725 214.98) (width 0.5) (layer F.Cu) (net 111))
-  (segment (start 349.755001 92.405001) (end 354.184001 92.405001) (width 0.5) (layer F.Cu) (net 111))
-  (segment (start 348.4 91.05) (end 349.755001 92.405001) (width 0.5) (layer F.Cu) (net 111))
-  (segment (start 316.544999 92.405001) (end 317.9 91.05) (width 0.5) (layer F.Cu) (net 111))
-  (segment (start 297.5 85.94) (end 297.5475 85.94) (width 0.5) (layer F.Cu) (net 111))
-  (segment (start 299.5 87.8925) (end 299.5 88.741998) (width 0.5) (layer F.Cu) (net 111))
-  (segment (start 297.5475 85.94) (end 299.5 87.8925) (width 0.5) (layer F.Cu) (net 111))
-  (segment (start 299.5 88.741998) (end 303.163003 92.405001) (width 0.5) (layer F.Cu) (net 111))
+  (segment (start 307.855001 92.405001) (end 316.544999 92.405001) (width 0.5) (layer F.Cu) (net 111))
   (segment (start 317.9 91.05) (end 348.4 91.05) (width 0.5) (layer F.Cu) (net 111))
-  (segment (start 303.163003 92.405001) (end 316.544999 92.405001) (width 0.5) (layer F.Cu) (net 111))
+  (segment (start 316.544999 92.405001) (end 317.9 91.05) (width 0.5) (layer F.Cu) (net 111))
+  (segment (start 348.4 91.05) (end 349.755001 92.405001) (width 0.5) (layer F.Cu) (net 111))
+  (segment (start 349.755001 92.405001) (end 354.184001 92.405001) (width 0.5) (layer F.Cu) (net 111))
+  (segment (start 301.39 85.94) (end 307.855001 92.405001) (width 0.5) (layer F.Cu) (net 111))
+  (segment (start 297.5 85.94) (end 301.39 85.94) (width 0.5) (layer F.Cu) (net 111))
   (segment (start 61.4 95.362998) (end 66.681099 100.644097) (width 0.25) (layer B.Cu) (net 112))
   (segment (start 61.4 80.3) (end 61.4 95.362998) (width 0.25) (layer B.Cu) (net 112))
@@
   (segment (start 315.345001 86.904999) (end 307.2 95.05) (width 0.25) (layer B.Cu) (net 216))
   (segment (start 300.7 95.05) (end 307.2 95.05) (width 0.25) (layer B.Cu) (net 216))
-  (segment (start 295.600009 84.049991) (end 296.25 83.4) (width 0.25) (layer B.Cu) (net 221))
-  (segment (start 296.25 83.4) (end 297.5 83.4) (width 0.25) (layer B.Cu) (net 221))
-  (segment (start 295.600009 86.649991) (end 295.600009 84.049991) (width 0.25) (layer B.Cu) (net 221))
-  (segment (start 292.4 89.85) (end 295.600009 86.649991) (width 0.25) (layer B.Cu) (net 221))
+  (segment (start 292.4 89.74) (end 292.4 89.85) (width 0.25) (layer B.Cu) (net 221))
+  (segment (start 293.099999 89.150001) (end 292.4 89.85) (width 0.25) (layer B.Cu) (net 221))
+  (segment (start 296.17499 86.07501) (end 293.099999 89.150001) (width 0.25) (layer B.Cu) (net 221))
+  (segment (start 296.17499 84.67751) (end 296.17499 86.07501) (width 0.25) (layer B.Cu) (net 221))
+  (segment (start 297.4525 83.4) (end 296.17499 84.67751) (width 0.25) (layer B.Cu) (net 221))
+  (segment (start 297.5 83.4) (end 297.4525 83.4) (width 0.25) (layer B.Cu) (net 221))
   (zone (net 1) (net_name GND) (layer F.Cu) (hatch edge 0.508)
     (connect_pads (clearance 0.508))

Commit message: Finish final PCB checks
Parts:
- moved D5 2.54 mm to (203.7, 63.3), turned to 180 degrees
Routing:
- net GND: track 153.4 -> 167.0 mm, vias 17 -> 16
- net +5V: track 596.5 -> 593.4 mm
- net Net-(F1-Pad2): track 24.5 -> 26.0 mm
- net Net-(D5-Pad1): track 81.3 -> 79.9 mm
