File: pcb/numpad_front/numpad_pcb.kicad_pcb (KiCad board)
At the start: 2 copper layers, 81 x 160.2 mm, 63 parts, among them J1 Conn_01x16_Female

Commit message: Revert freerouting
Parts:
- removed MOUNT1, MOUNT2, MOUNT3, MOUNT4, MOUNT5, MOUNT6, MOUNT7: MountingHole_2.2mm_M2_Pad, MountingHole:MountingHole_2.2mm_M2_Pad
- added REF**: MountingHole_2.2mm_M2_Pad, MountingHole:MountingHole_2.2mm_M2_Pad, F.Cu at (67.5, 30.0)
- added REF**: MountingHole_2.2mm_M2_Pad, MountingHole:MountingHole_2.2mm_M2_Pad, F.Cu at (68.4, 129.1)
- added REF**: MountingHole_2.2mm_M2_Pad, MountingHole:MountingHole_2.2mm_M2_Pad, F.Cu at (87.5, 167.1)
- added REF**: MountingHole_2.2mm_M2_Pad, MountingHole:MountingHole_2.2mm_M2_Pad, F.Cu at (135.0, 148.1)
- added REF**: MountingHole_2.2mm_M2_Pad, MountingHole:MountingHole_2.2mm_M2_Pad, F.Cu at (67.5, 87.0)
- added REF**: MountingHole_2.2mm_M2_Pad, MountingHole:MountingHole_2.2mm_M2_Pad, F.Cu at (140.6, 30.0)
Routing:
- net col19: track 152.8 -> 281.3 mm, vias 0 -> 1
- net col18: track 144.2 -> 253.9 mm, vias 0 -> 1
- net col17: track 119.0 -> 221.9 mm
- net LEDGND: track 371.9 -> 441.9 mm
- net row4: track 114.7 -> 78.5 mm
- net Net-(MX3-Pad3): track 66.0 -> 91.6 mm
- net Net-(MX7-Pad3): track 84.1 -> 104.3 mm
- net Net-(MX13-Pad3): track 126.0 -> 146.1 mm
- net +5V: track 110.9 -> 129.9 mm
- net Net-(MX11-Pad3): track 102.2 -> 120.1 mm
- net Net-(MX10-Pad3): track 107.9 -> 124.2 mm
- net Net-(MX14-Pad3): track 126.6 -> 140.6 mm
- net Net-(MX12-Pad3): track 132.7 -> 145.8 mm
- net Net-(MX9-Pad3): track 109.8 -> 121.7 mm
- net Net-(MX2-Pad3): track 64.8 -> 75.9 mm
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
Commit message: Finish PCB Silkscreen Decor
Parts:
- added G***: LOGO, silkscreens:numpad_decor, F.Cu at (100.8, 81.3)
- added REF**: MountingHole_2.2mm_M2_Pad, MountingHole:MountingHole_2.2mm_M2_Pad, F.Cu at (140.6, 87.0)
Other:
- board text added: "JLCJLCJLCJLC"
- board text added: "QBoard rev0 By QuantumManiac and Jlsajfj 2021-08-30 Numpad Board"
